File: ESP32C3 Mux/ESP32C3 Mux.kicad_sch (KiCad schematic)
At the start: 8 parts, among them J1 6130XX243121_613020243121, J2 Conn_01x02_Socket, U1 ESP32C3, U8 STLQ015M33R

Commit message: Re-layout of sensor control board
Connections:
- net SCL: now also U1.6 (D5); no longer U1.1 (D0)
- net SDA0: now also U1.5 (D4); no longer U1.2 (D1)
- net SDA1: now also U1.4 (D3); no longer U1.3 (D2)
- net SDA2: now also U1.3 (D2); no longer U1.4 (D3)
- net SDA3: now also U1.2 (D1); no longer U1.5 (D4)
- net SDA4: now also U1.1 (D0); no longer U1.6 (D5)
Changed lines of the file:
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@@
 		)
 	)
-	(label "SCL"
-		(at 193.04 119.38 0)
+	(label "SDA1"
+		(at 193.04 127 0)
 		(effects
 			(font
@@
 			)
 			(justify right bottom)
+		)
+	)
+	(label "SDA0"
+		(at 193.04 129.54 0)
+		(effects
+			(font
+				(size 1.27 1.27)
+			)
+			(justify left bottom)
 		)
 	)
@@
 		)
 	)
-	(label "SDA2"
-		(at 193.04 127 0)
+	(label "SCL"
+		(at 193.04 132.08 0)
 		(effects
 			(font
@@
 		)
 	)
-	(label "SDA3"
-		(at 193.04 129.54 0)
-		(effects
-			(font
-				(size 1.27 1.27)
-			)
-			(justify left bottom)
-		)
-	)
-	(label "SDA0"
-		(at 193.04 121.92 0)
+	(label "SDA4"
+		(at 193.04 119.38 0)
 		(effects
 			(font
@@
 		)
 	)
-	(label "SDA1"
+	(label "SDA2"
 		(at 193.04 124.46 0)
 		(effects
@@
 		)
 	)
-	(label "SDA4"
-		(at 193.04 132.08 0)
+	(label "SDA3"
+		(at 193.04 121.92 0)
 		(effects
 			(font
