File: ESP32C3 Mux/ESP32C3 Mux.kicad_pcb (KiCad board)
At the start: 2 copper layers, 28.7 x 28.9 mm, 4 parts, among them J1 6130XX243121_613020243121, U1 ESP32C3

Commit message: Final version
Parts:
- moved G*** 0.43 mm to (151.5, 122.9)
Routing:
- net GND: track 15.3 -> 18.2 mm, vias 21 -> 23
Other:
- outline, holes or cut-outs redrawn
Changed lines of the file:
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@@
 		(at 165.4683 116.1796 -90)
 		(property "Reference" "U1"
-			(at 8.4328 11.4935 180)
+			(at -8.6614 11.6205 180)
 			(layer "F.SilkS")
 			(effects
@@
 	(footprint "Electric-Feel:ntablogo"
 		(layer "F.Cu")
-		(at 151.0792 122.936)
+		(at 151.511 122.9106)
 		(property "Reference" "G***"
 			(at 0 0 0)
@@
 		(embedded_fonts no)
 	)
-	(gr_arc
-		(start 148.4376 126.3396)
-		(mid 147.71918 126.04202)
-		(end 147.4216 125.3236)
+	(gr_line
+		(start 176.2506 99.0092)
+		(end 176.2506 124.8664)
 		(stroke
 			(width 0.05)
@@
 	)
 	(gr_arc
-		(start 147.4216 98.4504)
-		(mid 147.71918 97.73198)
-		(end 148.4376 97.4344)
+		(start 149.0726 126.3904)
+		(mid 147.994969 125.944031)
+		(end 147.5486 124.8664)
 		(stroke
 			(width 0.05)
@@
 		(layer "Edge.Cuts")
 	)
-	(gr_arc
-		(start 176.1236 125.3236)
-		(mid 175.82602 126.04202)
-		(end 175.1076 126.3396)
+	(gr_line
+		(start 147.5486 124.8664)
+		(end 147.5486 99.0092)
 		(stroke
 			(width 0.05)
@@
 	)
 	(gr_line
-		(start 148.4376 97.4344)
-		(end 175.1076 97.4344)
+		(start 149.0726 97.4852)
+		(end 174.7266 97.4852)
 		(stroke
 			(width 0.05)
@@
 		(layer "Edge.Cuts")
 	)
-	(gr_line
-		(start 175.1076 126.3396)
-		(end 148.4376 126.3396)
+	(gr_arc
+		(start 176.2506 124.8664)
+		(mid 175.804231 125.944031)
+		(end 174.7266 126.3904)
 		(stroke
 			(width 0.05)
@@
 	)
 	(gr_line
-		(start 176.1236 98.4504)
-		(end 176.1236 125.3236)
+		(start 174.7266 126.3904)
+		(end 149.0726 126.3904)
+		(stroke
+			(width 0.05)
+			(type default)
+		)
+		(layer "Edge.Cuts")
+	)
+	(gr_arc
+		(start 174.7266 97.4852)
+		(mid 175.804231 97.931569)
+		(end 176.2506 99.0092)
+		(stroke
+			(width 0.05)
+			(type default)
+		)
+		(layer "Edge.Cuts")
+	)
+	(gr_arc
+		(start 147.5486 99.0092)
+		(mid 147.994969 97.931569)
+		(end 149.0726 97.4852)
 		(stroke
 			(width 0.05)
@@
 		(layer "Edge.Cuts")
 	)
-	(gr_arc
-		(start 175.1076 97.4344)
-		(mid 175.82602 97.73198)
-		(end 176.1236 98.4504)
-		(stroke
-			(width 0.05)
-			(type default)
-		)
-		(layer "Edge.Cuts")
-	)
-	(gr_line
-		(start 147.4216 125.3236)
-		(end 147.4216 98.4504)
-		(stroke
-			(width 0.05)
-			(type default)
-		)
-		(layer "Edge.Cuts")
-	)
 	(segment
 		(start 150.1648 101.3968)
@@
 	)
 	(segment
-		(start 167.9448 122.7836)
-		(end 158.8008 113.6396)
-		(width 0.2)
-		(layer "F.Cu")
-		(net 1)
-	)
-	(segment
 		(start 157.7848 101.3968)
 		(end 160.3248 101.3968)
@@
 	)
 	(segment
-		(start 158.8008 113.6396)
-		(end 158.8008 107.3404)
+		(start 158.496 107.0356)
+		(end 158.496 106.1212)
 		(width 0.2)
 		(layer "F.Cu")
@@
 	)
 	(segment
-		(start 158.8008 107.3404)
-		(end 158.496 107.0356)
+		(start 159.0548 113.8936)
+		(end 159.0548 107.5944)
+		(width 0.2)
+		(layer "F.Cu")
+		(net 1)
+	)
+	(segment
+		(start 167.9448 122.7836)
+		(end 159.0548 113.8936)
+		(width 0.2)
+		(layer "F.Cu")
+		(net 1)
+	)
+	(segment
+		(start 167.9448 123.7996)
+		(end 167.9448 122.7836)
 		(width 0.2)
 		(layer "F.Cu")
@@
 	)
 	(segment
-		(start 167.9448 123.7996)
-		(end 167.9448 122.7836)
-		(width 0.2)
-		(layer "F.Cu")
-		(net 1)
-	)
-	(segment
-		(start 158.496 107.0356)
-		(end 158.496 106.1212)
-		(width 0.2)
-		(layer "F.Cu")
-		(net 1)
-	)
-	(segment
 		(start 149.0083 102.5533)
 		(end 149.0083 104.8631)
@@
 	)
 	(segment
+		(start 159.0548 107.5944)
+		(end 158.496 107.0356)
+		(width 0.2)
+		(layer "F.Cu")
+		(net 1)
+	)
+	(segment
 		(start 165.4556 101.3968)
 		(end 166.3192 100.5332)
@@
 	)
 	(segment
+		(start 170.4848 123.7996)
+		(end 171.4246 124.7394)
+		(width 0.254)
+		(layer "F.Cu")
+		(net 2)
+	)
+	(segment
 		(start 170.4848 101.3968)
 		(end 171.3484 100.5332)
@@
 		(start 173.0248 101.3968)
 		(end 172.1104 102.3112)
+		(width 0.254)
+		(layer "F.Cu")
+		(net 2)
+	)
+	(segment
+		(start 170.4848 123.7996)
+		(end 169.3418 122.6566)
 		(width 0.254)
 		(layer "F.Cu")
@@
 	)
 	(via
+		(at 171.4246 124.7394)
+		(size 0.6)
+		(drill 0.3)
+		(layers "F.Cu" "B.Cu")
+		(net 2)
+	)
+	(via
 		(at 163.7284 100.5332)
 		(size 0.6)
@@
 	)
 	(via
+		(at 169.3418 122.6566)
+		(size 0.6)
+		(drill 0.3)
+		(layers "F.Cu" "B.Cu")
+		(net 2)
+	)
+	(via
 		(at 166.3192 100.5332)
 		(size 0.6)
@@
 		(polygon
 			(pts
-				(xy 146.3548 96.7076) (xy 177.6548 96.7076) (xy 177.6548 126.2092) (xy 146.3548 126.2092)
-			)
-		)
+				(xy 146.3548 96.7076) (xy 177.6548 96.7076) (xy 177.6548 127.2506) (xy 146.3548 127.2506)
+			)
+		)
